File: MicroUSB.sch (KiCad schematic (older format))
At the start: 11 parts, among them J1 USB_OTG, J2 Conn_01x05, Q1 MMBT3904, U1 USBLC6-2SC6

Commit message: Re-designed (using non-handsolder footprint)
Parts:
- R1, R2, R3, R4, R5, R6, R7: footprint Resistors_SMD:R_0603_HandSoldering -> Resistors_SMD:R_0603
- U1: footprint TO_SOT_Packages_SMD:SOT-23-6_Handsoldering -> TO_SOT_Packages_SMD:SOT-23-6
Changed lines of the file:
@@
 F 0 "R3" V 2950 3750 50  0000 C CNN
 F 1 "20R" V 2950 3600 50  0000 C CNN
-F 2 "Resistors_SMD:R_0603_HandSoldering" V 2880 3600 50  0001 C CNN
+F 2 "Resistors_SMD:R_0603" V 2880 3600 50  0001 C CNN
 F 3 "" H 2950 3600 50  0001 C CNN
 	1    2950 3600
@@
 F 0 "R1" V 2950 3550 50  0000 C CNN
 F 1 "1k5" V 2950 3400 50  0000 C CNN
-F 2 "Resistors_SMD:R_0603_HandSoldering" V 2880 3400 50  0001 C CNN
+F 2 "Resistors_SMD:R_0603" V 2880 3400 50  0001 C CNN
 F 3 "" H 2950 3400 50  0001 C CNN
 	1    2950 3400
@@
 F 0 "R2" V 2950 3650 50  0000 C CNN
 F 1 "20R" V 2950 3500 50  0000 C CNN
-F 2 "Resistors_SMD:R_0603_HandSoldering" V 2880 3500 50  0001 C CNN
+F 2 "Resistors_SMD:R_0603" V 2880 3500 50  0001 C CNN
 F 3 "" H 2950 3500 50  0001 C CNN
 	1    2950 3500
@@
 F 0 "R5" V 3680 2800 50  0000 C CNN
 F 1 "10K" V 3600 2800 50  0000 C CNN
-F 2 "Resistors_SMD:R_0603_HandSoldering" V 3530 2800 50  0001 C CNN
+F 2 "Resistors_SMD:R_0603" V 3530 2800 50  0001 C CNN
 F 3 "" H 3600 2800 50  0001 C CNN
 	1    3600 2800
@@
 F 0 "R6" V 3700 3300 50  0000 C CNN
 F 1 "36k" V 3600 3300 50  0000 C CNN
-F 2 "Resistors_SMD:R_0603_HandSoldering" V 3530 3300 50  0001 C CNN
+F 2 "Resistors_SMD:R_0603" V 3530 3300 50  0001 C CNN
 F 3 "" H 3600 3300 50  0001 C CNN
 	1    3600 3300
@@
 F 0 "R4" V 2950 3850 50  0000 C CNN
 F 1 "100k" V 3050 3700 50  0000 C CNN
-F 2 "Resistors_SMD:R_0603_HandSoldering" V 2880 3700 50  0001 C CNN
+F 2 "Resistors_SMD:R_0603" V 2880 3700 50  0001 C CNN
 F 3 "" H 2950 3700 50  0001 C CNN
 	1    2950 3700
@@
 F 0 "R7" V 3980 3100 50  0000 C CNN
 F 1 "100R" V 3900 3100 50  0000 C CNN
-F 2 "Resistors_SMD:R_0603_HandSoldering" V 3830 3100 50  0001 C CNN
+F 2 "Resistors_SMD:R_0603" V 3830 3100 50  0001 C CNN
 F 3 "" H 3900 3100 50  0001 C CNN
 	1    3900 3100
@@
 F 0 "U1" H 4300 3550 60  0000 C CNN
 F 1 "USBLC6-2SC6" H 4350 4050 60  0000 C CNN
-F 2 "TO_SOT_Packages_SMD:SOT-23-6_Handsoldering" H 4400 3700 60  0001 C CNN
+F 2 "TO_SOT_Packages_SMD:SOT-23-6" H 4400 3700 60  0001 C CNN
 F 3 "" H 4400 3700 60  0001 C CNN
 	1    4400 3700
